Commit message: avanzando

File: urdf/ebamk2.xacro (robot description, xacro)
@@ -36,5 +36,5 @@
       <origin xyz="0 0 0" rpy="0 0 0"/>
       <!-- <mass value="0.058"/> -->
-      <mass value="0.19357368"/>
+      <mass value="1.9357368"/>
       <!-- <inertia ixx="1.429e-4"  ixy="2.778e-10"  ixz="1.773e-8" iyy="1.943e-4" iyz="-2.656e-7" izz="5.361e-5" /> -->
       <inertia ixx="1.84569610e-4"  ixy="-4.09475462e-6"  ixz="-2.91063667e-5" iyy="7.65700035e-4" iyz="2.32776537e-8" izz="9.00861891e-4" />
@@ -194,5 +194,5 @@
       <origin xyz="0 0 0" rpy="0 0 0"/>
       <!-- <mass value="0.058"/> -->
-      <mass value="0.19357368"/>
+      <mass value="0.09357368"/>
       <!-- <inertia ixx="1.429e-4"  ixy="2.778e-10"  ixz="1.773e-8" iyy="1.943e-4" iyz="-2.656e-7" izz="5.361e-5" /> -->
       <inertia ixx="1.84569610e-4"  ixy="-4.09475462e-6"  ixz="-2.91063667e-5" iyy="7.65700035e-4" iyz="2.32776537e-8" izz="9.00861891e-4" />
