Commit message: se configuran los controladores de manera correcta

File: urdf/ebamk2-complete.xacro (robot description, xacro)
@@ -2,5 +2,5 @@
 <robot name="ebamk2" xmlns:xacro="http://www.ros.org/wiki/xacro">
  <xacro:include filename="$(find eezybot)/urdf/gazebo.xacro" />
-  <!--xacro:ros_control prefix=""/-->
+ <xacro:ros_control prefix="/"/>
   <xacro:macro name="cuboid_inertia_def" params="x y z mass">
     <inertia
@@ -10,7 +10,12 @@
       ixy="0.0" iyz="0.0" ixz="0.0"/>
   </xacro:macro>
-<link name="base_link">
- </link>
+<link name="world"/>
+<link name="base_link"/>
 <!-- BASE LINK -->
+  <joint name="fixed" type="fixed">
+    <parent link="world"/>
+    <child link="base_link"/>
+    <origin xyz="0 0 0" rpy="0 0 0" />
+  </joint>
   <link
     name="link_0">
@@ -32,6 +37,6 @@
     <inertial>
       <origin xyz="0 0 0.0275" rpy="0 0 0"/>
-      <mass value="2"/>
-      <xacro:cuboid_inertia_def x="0.055" y="0.055" z="0.055" mass="2"/>
+      <mass value="5"/>
+      <xacro:cuboid_inertia_def x="0.055" y="0.055" z="0.055" mass="5"/>
     </inertial>
   </link>
@@ -47,5 +52,5 @@
     <child link="link_1" />
     <axis xyz="0 0 1" />
-    <limit effort="0" velocity="0"
+    <limit effort="10" velocity="0.50"
       lower="-0.7854" upper="0.7854"/>
   </joint>
@@ -82,5 +87,5 @@
     <child link="link_2" />
     <axis xyz="0 0 1" />
-    <limit effort="0" velocity="0"
+    <limit effort="10" velocity="0.40"
       lower="-0.80" upper="0.35"/>
   </joint>
@@ -109,5 +114,5 @@
   </link>
   <!-- VIRTUAL MIMIC JOINT 2-->
-  <joint name="joint2v" type="revolute">
+  <!--joint name="joint2v" type="revolute">
     <origin xyz="-0.021 0.135 -0.0105" rpy="1.570796325 0 0" />
     <parent link="link_2"/>
@@ -116,36 +121,22 @@
     <limit effort="30" velocity="1.0" lower="-3.14159" upper="3.14159" />
     <mimic joint="joint_2" multiplier="-1" offset="0" />
-  </joint>
-  <link name="link_2v">
-    <visual>
-      <geometry>
-        <cylinder length="0.001" radius="0.0001"/>
-      </geometry>
-      <material name="">
-        <color rgba="0 0 0 0" />
-      </material>
-      <origin rpy="0 0 0" xyz="0 0 0"/>
-    </visual>
-    <collision>
-      <geometry>
-        <cylinder length="0.0001" radius="0.0001"/>
-      </geometry>
-      <origin rpy="0 0 0" xyz="0 0 0"/>
-    </collision>
-    <!--inertial>
-      <origin xyz="0 0 0" rpy="0 0 0"/>
-      <mass value="0.0015"/>
-      <xacro:cuboid_inertia_def x="0.0001" y="0.0002" z="0.0005" mass="0.0015"/>
-    </inertial-->
-  </link>
+  </joint-->
+  <joint name="joint_3" type="revolute">
+    <origin xyz="-0.021 0.135 -0.0105" rpy="1.570796325 0 0" />
+    <parent link="link_2"/>
+    <child link="link_3"/>
+    <axis xyz="0 1 0"/>
+    <limit effort="30" velocity="0.5" lower="${-0.49}" upper="1.22" />
+    <!--mimic joint="joint_2" multiplier="-1" offset="0" /-->
+  </joint>
 <!-- JOINT 3 ELBOW -->
-  <joint name="joint_3" type="revolute">
+  <!--joint name="joint_3" type="revolute">
     <origin xyz="0 0 0" rpy="0 0 0" />
-    <parent link="link_2" />
+    <parent link="link_2v" />
     <child link="link_3" />
     <axis xyz="0 1 0" />
     <limit effort="0" velocity="0"
       lower="-0.77" upper="0.45"/>
-  </joint>
+  </joint-->
 <!-- LINK 3 ELBOW -->
    <link name="link_3">
@@ -177,5 +168,5 @@
     <child link="link_4" />
     <axis xyz="0 1 0" />
-    <limit effort="0" velocity="0" lower="-3.14159" upper="3.14159"/>
+    <limit effort="10" velocity="0.4" lower="-0.5" upper="1"/>
     <!--<mimic joint="joint_3" multiplier="1" offset="0" />-->
   </joint>
@@ -287,12 +278,12 @@
     </inertial>
   </link>
-  <!-- TRANSMISSIONS -->
+<!-- TRANSMISSIONS -->
   <transmission name="trans_1">
     <type>transmission_interface/SimpleTransmission</type>
     <joint name="joint_1">
-      <hardwareInterface>PositionJointInterface</hardwareInterface>
+      <hardwareInterface>EffortJointInterface</hardwareInterface>
     </joint>
     <actuator name="servo1">
-      <hardwareInterface>PositionJointInterface</hardwareInterface>
+      <hardwareInterface>EffortJointInterface</hardwareInterface>
       <mechanicalReduction>1</mechanicalReduction>
     </actuator>
@@ -301,8 +292,8 @@
     <type>transmission_interface/SimpleTransmission</type>
     <joint name="joint_2">
-      <hardwareInterface>PositionJointInterface</hardwareInterface>
+      <hardwareInterface>EffortJointInterface</hardwareInterface>
     </joint>
     <actuator name="servo2">
-      <hardwareInterface>PositionJointInterface</hardwareInterface>
+      <hardwareInterface>EffortJointInterface</hardwareInterface>
       <mechanicalReduction>1</mechanicalReduction>
     </actuator>
@@ -311,18 +302,18 @@
     <type>transmission_interface/SimpleTransmission</type>
     <joint name="joint_3">
-      <hardwareInterface>PositionJointInterface</hardwareInterface>
+      <hardwareInterface>EffortJointInterface</hardwareInterface>
     </joint>
     <actuator name="servo3">
-      <hardwareInterface>PositionJointInterface</hardwareInterface>
+      <hardwareInterface>EffortJointInterface</hardwareInterface>
       <mechanicalReduction>1</mechanicalReduction>
     </actuator>
   </transmission>
-  <transmission name="trans_6">
+  <transmission name="trans_4">
     <type>transmission_interface/SimpleTransmission</type>
-    <joint name="joint_6">
-      <hardwareInterface>PositionJointInterface</hardwareInterface>
+    <joint name="joint_4">
+      <hardwareInterface>EffortJointInterface</hardwareInterface>
     </joint>
     <actuator name="servo4">
-      <hardwareInterface>PositionJointInterface</hardwareInterface>
+      <hardwareInterface>EffortJointInterface</hardwareInterface>
       <mechanicalReduction>1</mechanicalReduction>
     </actuator>

Commit message: se divide gazebo en spawn y gazebo. Se arreglan las inercias y se reducen las geometrias de colision a solidos simples

File: urdf/ebamk2-complete.xacro (robot description, xacro)
@@ -30,7 +30,7 @@
     </visual>
     <collision>
-      <origin xyz="0 0 0" rpy="0 0 0" />
-      <geometry>
-        <mesh filename="package://eezybot/meshes/base_link.STL" />
+      <origin xyz="0 0 0.0275" rpy="0 0 0" />
+      <geometry>
+        <box size="0.055 0.055 0.055"/>
       </geometry>
     </collision>
@@ -70,7 +70,7 @@
     <collision>
       <origin
-        xyz="0 -0.04 0" rpy="0 0 0" />
-      <geometry>
-        <mesh filename="package://eezybot/meshes/link_1.STL" />
+        xyz="0 0 0.04" rpy="0 0 0" />
+      <geometry>
+        <box size="0.032 0.052 0.0415"/>
       </geometry>
     </collision>
@@ -102,11 +102,11 @@
     </visual>
     <collision>
-      <origin xyz="0 0 0.0075" rpy="3.14159 0 0" />
-      <geometry>
-        <mesh filename="package://eezybot/meshes/link_2.STL" />
-      </geometry>
-    </collision>
-    <inertial>
-      <origin xyz="0 0.0675 0.0075" rpy="3.14159 0 0"/>
+      <origin xyz="${(-0.021-0)/2.0} ${(0.135+0.005)/2.0} ${0.02+(-0.0105-0.037)/2.0}" rpy="3.14159 0 ${0.14888994}" />
+      <geometry>
+        <box size="${0.01} ${0.135+0.005} ${0.01}"/>
+      </geometry>
+    </collision>
+    <inertial>
+      <origin xyz="${(-0.021-0)/2.0} ${(0.135+0.005)/2.0} ${0.02+(-0.0105-0.037)/2.0}" rpy="3.14159 0 ${0.14888994}" />
       <mass value="0.12"/>
       <xacro:cuboid_inertia_def x="0.01" y="0.135" z="0.01" mass="0.12"/>
@@ -151,13 +151,13 @@
     </visual>
     <collision>
-      <origin xyz="0 0.0335  0.002" rpy="1.570796325 0 0" />
-      <geometry>
-        <mesh filename="package://eezybot/meshes/link_3.STL" />
-      </geometry>
-    </collision>
-    <inertial>
-      <origin xyz="0.075 0.00 0" rpy="1.570796325 0 0" />
+      <origin xyz="${(0.1459)/2.0} ${(0.0203)/2.0} ${0.0185/2.}" rpy="1.570796325 ${-0.126126098371} 0" />
+      <geometry>
+        <box size="${0.1459} 0.01 0.01" />
+      </geometry>
+    </collision>
+    <inertial>
+      <origin xyz="${(0.1459)/2.0} ${(0.0203)/2.0} ${0.0185/2.}" rpy="1.570796325 ${-0.126126098371} 0" />
       <mass value="0.07"/>
-      <xacro:cuboid_inertia_def x="0.205" y="0.01" z="0.01" mass="0.07"/>
+      <xacro:cuboid_inertia_def x="0.1459" y="0.01" z="0.01" mass="0.07"/>
     </inertial>
   </link>
@@ -183,13 +183,13 @@
     </visual>
     <collision>
-      <origin xyz="-0.006 0 -0.0394" rpy="0 0 0" />
-      <geometry>
-        <mesh filename="package://eezybot/meshes/link_4.STL" scale="0.001 0.001 0.001" />
-      </geometry>
-    </collision>
-    <inertial>
-      <origin xyz="0 0 0" rpy="0 0 0" />
+      <origin xyz="0.015 0.015 -0.02" rpy="0 0 0" />
+      <geometry>
+        <box size="0.03 0.03 0.04" />
+      </geometry>
+    </collision>
+    <inertial>
+      <origin xyz="0.015 0.015 -0.02" rpy="0 0 0" />
       <mass value="0.03"/>
-      <xacro:cuboid_inertia_def x="0.01" y="0.03" z="0.01" mass="0.03"/>
+      <xacro:cuboid_inertia_def x="0.03" y="0.03" z="0.04" mass="0.03"/>
     </inertial>
   </link>

Commit message: se agrega joint del gripper. Falta agregar un mimicplugin

File: urdf/ebamk2-complete.xacro (robot description, xacro)
@@ -230,5 +230,5 @@
     <child link="claw_l"/>
     <axis xyz="0 0 1" />
-    <limit effort="0" lower="0" upper="0.65" velocity="1.0" />
+    <limit effort="10" lower="0" upper="0.65" velocity="1.0" />
   </joint>
   <joint name="joint_7" type="revolute">
@@ -254,5 +254,5 @@
     </collision>
     <inertial>
-      <origin xyz="0.00 0.000 0" rpy="0 0 2.9" />
+      <origin xyz="0.0235 0.000 0" rpy="0 0 2.9" />
       <mass value="0.01"/>
       <xacro:cuboid_inertia_def x="0.047" y="0.005" z="0.005" mass="0.01"/>
@@ -319,3 +319,13 @@
     </actuator>
   </transmission>
+    <transmission name="trans_6">
+    <type>transmission_interface/SimpleTransmission</type>
+    <joint name="joint_6">
+      <hardwareInterface>EffortJointInterface</hardwareInterface>
+    </joint>
+    <actuator name="servo6">
+      <hardwareInterface>EffortJointInterface</hardwareInterface>
+      <mechanicalReduction>1</mechanicalReduction>
+    </actuator>
+  </transmission>
 </robot>
